Commit message: Hokuyo and camera sensors added

File: rugved_description/urdf/rugved_description.urdf (robot description, URDF)
Before this commit: robot rugved_description, 5 links, 4 joints
Links:
- added link camera_link, mass 1e-5; collision box size=0.08 0.08 0.08; visual box size=0.08 0.08 0.08
- added link hokuyo_link, mass 1e-5; collision box size=0.1 0.1 0.1; visual box size=0.1 0.1 0.1
Joints:
- added joint camera_joint: type fixed, parent base_link, child camera_link, origin xyz=0.38 -0.00022 0.45 rpy=0 0 0, axis 0 1 0
- added joint hokuyo_joint: type fixed, parent base_link, child hokuyo_link, origin xyz=0.38 -0.00022 0.7 rpy=0 0 0, axis 0 1 0
